Commit message: feat: expand radar coverage to 6 panels — zero gap 360°
xacro:
- radar_h_fov: 55° → 60° (AWR1843 realistic, tiles exactly at 60° spacing)
- Panels A-F at 0°/60°/120°/180°/240°/300° — one per hexacopter arm
- Add panels E (240°) and F (300°): links, joints, sensor plugins, materials
- m_rbox: 0.750 → 0.860 kg (+2× AWR1843 mass)
- Link/joint count: 68/67 → 72/71

isr_lidar_mpc.py:
- _RADAR_TOPICS: add panels E and F with env-var overrides
- _PANEL_YAWS_DEG: 4-panel {B:270,C:180,D:90} → 6-panel 60° grid
- _discover_radar_topics: scan for E and F in addition to A-D

Coverage: 4×55°=220° with 35° gaps → 6×60°=360°, zero gaps

Co-Authored-By: Claude Sonnet 4.6 <noreply@anthropic.com>

File: new_drone/mbc3_radar_drone.xacro (robot description, xacro)
@@ -10,10 +10,10 @@
   ROS         : ROS2 Jazzy + Gazebo Harmonic (gz-sim 8.x)
   Units       : SI (metres, kg, radians, seconds)
-  Structure   : 68 links, 67 joints
+  Structure   : 72 links, 71 joints
   Geometry    : Multi-body realistic visuals per component
   Physics     : Correct inertia tensors, Gazebo mu/kp/kd, damping
   Sensors     : IMU 400Hz (VN-100), GPS/GNSS 10Hz (Here3+),
                 Barometer 50Hz, Magnetometer 50Hz,
-                Optical-flow 60Hz, 4× FMCW Radar panels 10Hz
+                Optical-flow 60Hz, 6× FMCW Radar panels 10Hz
   Control     : ros2_control gz_ros2_control::GazeboSimSystem
                 VelocityJointInterface × 6 motors
@@ -119,6 +119,7 @@
   <xacro:property name="panel_arm_off"  value="${0.110*viz_scale}"/>
   <xacro:property name="radome_t"       value="${0.005*viz_scale}"/>
-  <!-- 24 GHz FMCW: ±27.5° H-FOV, ±22.5° V-FOV per panel -->
-  <xacro:property name="radar_h_fov"    value="${55.0*D2R}"/>
+  <!-- 24 GHz FMCW: ±30° H-FOV, ±22.5° V-FOV per panel.
+       6 panels at 60° spacing × 60° FOV = seamless 360° coverage, zero gaps. -->
+  <xacro:property name="radar_h_fov"    value="${60.0*D2R}"/>
   <xacro:property name="radar_v_fov"    value="${45.0*D2R}"/>
   <xacro:property name="radar_range_min" value="2.0"/>
@@ -158,5 +159,5 @@
   <xacro:property name="m_plate"        value="0.070"/>
   <xacro:property name="m_so"           value="0.010"/>
-  <xacro:property name="m_rbox"         value="0.750"/>  <!-- Al shell + AWR1843×4 + Doodle Labs + Jetson Orin NX + misc -->
+  <xacro:property name="m_rbox"         value="0.860"/>  <!-- Al shell + AWR1843×6 + Doodle Labs + Jetson Orin NX + misc -->
   <xacro:property name="m_panel"        value="0.055"/>
   <xacro:property name="m_bat"          value="1.050"/>  <!-- 6S 10000mAh single pack -->
@@ -1373,14 +1374,17 @@
   <xacro:standoff id="rl" px="${-so_pcd}" py=" ${so_pcd}"/>
   <xacro:standoff id="rr" px="${-so_pcd}" py="${-so_pcd}"/>
-  <!-- 4 antenna panels.
-       Panel faces (radar_frame +X):
-         A → +X (forward),  B → −Y (right, FLU convention),
-         C → −X (rear),     D → +Y (left)
-       Fusion node panel_yaws must match:
-         A=0, B=−π/2, C=π, D=+π/2                          -->
+  <!-- 6 antenna panels at 60° spacing — one per arm (hex layout).
+       Panel faces (radar_frame +X), FLU convention:
+         A →   0° (forward)       D → 180° (rear)
+         B →  60° (fwd-left)      E → 240° (rear-right)
+         C → 120° (rear-left)     F → 300° (fwd-right)
+       6 × 60° FOV = seamless 360° coverage, zero gaps.
+       Fusion node panel_yaws must match these angles.       -->
   <xacro:antenna_panel id="A" angle_deg="0"/>
-  <xacro:antenna_panel id="B" angle_deg="270"/>
-  <xacro:antenna_panel id="C" angle_deg="180"/>
-  <xacro:antenna_panel id="D" angle_deg="90"/>
+  <xacro:antenna_panel id="B" angle_deg="60"/>
+  <xacro:antenna_panel id="C" angle_deg="120"/>
+  <xacro:antenna_panel id="D" angle_deg="180"/>
+  <xacro:antenna_panel id="E" angle_deg="240"/>
+  <xacro:antenna_panel id="F" angle_deg="300"/>
   <!-- 2 landing gear sets -->
   <xacro:landing_gear side="L" y_sign=" 1"/>
@@ -1639,7 +1643,8 @@
   <!-- ── Radar panel sensors — gpu_lidar for GPU ray-casting ─ -->
   <!-- Using gpu_lidar gives 10–50× better performance vs cpu ray.
-       Horizontal: 220 samples over ±radar_h_fov = 55° total.
-       Vertical:    90 samples over ±radar_v_fov = 45° total.
-       Range 0.5–5000 m, Gaussian noise σ=0.8 m (FMCW range error). -->
+       Horizontal: 220 samples over radar_h_fov = 60° total (±30°).
+       Vertical:    90 samples over radar_v_fov = 45° total (±22.5°).
+       Range 0.5–5000 m, Gaussian noise σ=0.8 m (FMCW range error).
+       6 panels × 60° = seamless 360° coverage.                     -->
   <xacro:macro name="radar_sensor_plugin" params="id">
     <gazebo reference="radar_frame_${id}">
@@ -1682,4 +1687,6 @@
   <xacro:radar_sensor_plugin id="C"/>
   <xacro:radar_sensor_plugin id="D"/>
+  <xacro:radar_sensor_plugin id="E"/>
+  <xacro:radar_sensor_plugin id="F"/>
   <!-- ── Optical flow: downward-facing rangefinder + camera ── -->
   <gazebo reference="optical_flow_link">
@@ -1807,4 +1814,6 @@
   <gazebo reference="antenna_panel_C"><material>Gazebo/WoodPallet</material></gazebo>
   <gazebo reference="antenna_panel_D"><material>Gazebo/WoodPallet</material></gazebo>
+  <gazebo reference="antenna_panel_E"><material>Gazebo/WoodPallet</material></gazebo>
+  <gazebo reference="antenna_panel_F"><material>Gazebo/WoodPallet</material></gazebo>
 <!-- ═══════════════════════════════════════════════════════════════
      SECTION 17 — PX4 GAZEBO HARMONIC MOTOR CONTROL

Commit message: fix: stabilise mbc3_radar_drone SITL flight — 6 SDF/airframe bugs
B7-1: gpu_lidar -> lidar for radar A-F + rangefinder (no GPU in SITL)
B7-2: remove robotNamespace from MulticopterMotorModel plugins
      (hardcoded 'mbc3_radar_drone' != spawned 'mbc3_radar_drone_0')
B7-3: remove 6x LiftDrag plugins from motor_bell links
      (double thrust with MulticopterMotorModel -> violent overcorrection)
B7-4: set all motor joint axes to 0 0 1 (was 0 0 -1 for CW motors)
      (drag torque double-negation caused partial yaw sign error)
B7-5: invert CA_ROTOR KM signs to match x500/Gazebo convention
      (CCW=+0.05, CW=-0.05; was reversed -> yaw positive feedback loop)
B7-6: MPC_THR_HOVER 0.72 -> 0.63 (empirical from hover_thrust_estimate)

Result: CCW/CW motor ratio 1.9x -> 1.00x, yaw rate 8.4 -> 0.09 rad/s,
attitude +-43deg -> +-4deg. Drone reaches 2.4m hover stably.
Log: 2026-05-19/13_58_15.ulg

Co-Authored-By: Claude Sonnet 4.6 <noreply@anthropic.com>

File: new_drone/mbc3_radar_drone.xacro (robot description, xacro)
@@ -123,5 +123,5 @@
   <xacro:property name="radar_h_fov"    value="${60.0*D2R}"/>
   <xacro:property name="radar_v_fov"    value="${45.0*D2R}"/>
-  <xacro:property name="radar_range_min" value="2.0"/>
+  <xacro:property name="radar_range_min" value="0.5"/>
   <xacro:property name="radar_range_max" value="5000.0"/>
   <xacro:property name="radar_res"      value="0.120"/>
@@ -1595,5 +1595,5 @@
           <noise type="gaussian">
             <mean>0.0</mean>
-            <stddev>0.1</stddev>   <!-- ±0.1 m typical MEMS baro -->
+            <stddev>0.2</stddev>   <!-- ±0.2 m outdoor MEMS baro without wind model -->
           </noise>
         </vertical_position>
@@ -1654,5 +1654,6 @@
         <visualize>false</visualize>
         <topic>${tp}/radar_${id}/scan</topic>
-        <ray>
+        <!-- gpu_lidar requires <lidar> block, not <ray> (Gazebo Harmonic) -->
+        <lidar>
           <scan>
             <horizontal>
@@ -1677,7 +1678,7 @@
             <type>gaussian</type>
             <mean>0.0</mean>
-            <stddev>0.8</stddev>
+            <stddev>0.10</stddev>  <!-- reduced from 0.8: σ≈0.83× resolution (0.12m) -->
           </noise>
-        </ray>
+        </lidar>
       </sensor>
     </gazebo>
@@ -1692,9 +1693,11 @@
   <gazebo reference="optical_flow_link">
     <!-- Rangefinder (TFmini-equivalent) for altitude hold -->
-    <sensor name="rangefinder" type="ray">
+    <!-- type=gpu_lidar + <lidar> block required for Gazebo Harmonic; type=ray is deprecated -->
+    <sensor name="rangefinder" type="gpu_lidar">
       <always_on>true</always_on>
       <update_rate>60</update_rate>
+      <visualize>false</visualize>
       <topic>${tp}/rangefinder/range</topic>
-      <ray>
+      <lidar>
         <scan>
           <horizontal>
@@ -1715,5 +1718,5 @@
           <stddev>0.005</stddev>
         </noise>
-      </ray>
+      </lidar>
     </sensor>
     <!-- Optical flow camera -->
@@ -1721,4 +1724,5 @@
       <always_on>true</always_on>
       <update_rate>60</update_rate>
+      <visualize>false</visualize>
       <topic>${tp}/optical_flow/image_raw</topic>
       <camera>
@@ -1737,6 +1741,11 @@
        Model-level plugin block avoids urdf2sdf placing plugin
        inside <link> element (which triggers SDF warning).    -->
-  <xacro:macro name="rotor_aero" params="num link_name spin_dir">
-    <gazebo reference="${link_name}">
+  <!-- LiftDrag must reference the actual spinning link (motor_bell_N), not prop_N.
+       prop_N is a fixed-joint child and may be merged in SDF; motor_bell_N is the
+       continuous joint child and is guaranteed to survive as a physics link.
+       <forward> is always 1 0 0: yaw torque direction is set by momentConstant sign
+       in the motor model — reversing <forward> per CW/CCW doubles torque error. -->
+  <xacro:macro name="rotor_aero" params="num">
+    <gazebo reference="motor_bell_${num}">
       <plugin filename="gz-sim-lift-drag-system"
               name="gz::sim::systems::LiftDrag">
@@ -1752,17 +1761,16 @@
         <area>${PI*prop_r*prop_r}</area>
         <air_density>1.2041</air_density>
-        <forward>${spin_dir} 0 0</forward>
+        <forward>1 0 0</forward>
         <upward>0 0 1</upward>
-        <link_name>${link_name}</link_name>
+        <link_name>motor_bell_${num}</link_name>
       </plugin>
     </gazebo>
   </xacro:macro>
-  <!-- Forward vectors alternate with spin direction -->
-  <xacro:rotor_aero num="0" link_name="prop_0" spin_dir=" 1"/>
-  <xacro:rotor_aero num="1" link_name="prop_1" spin_dir="-1"/>
-  <xacro:rotor_aero num="2" link_name="prop_2" spin_dir=" 1"/>
-  <xacro:rotor_aero num="3" link_name="prop_3" spin_dir="-1"/>
-  <xacro:rotor_aero num="4" link_name="prop_4" spin_dir=" 1"/>
-  <xacro:rotor_aero num="5" link_name="prop_5" spin_dir="-1"/>
+  <xacro:rotor_aero num="0"/>
+  <xacro:rotor_aero num="1"/>
+  <xacro:rotor_aero num="2"/>
+  <xacro:rotor_aero num="3"/>
+  <xacro:rotor_aero num="4"/>
+  <xacro:rotor_aero num="5"/>
   <!-- ── Landing skid contact surface tuning ─────────────── -->
   <gazebo reference="lg_skid_L">
@@ -1839,5 +1847,5 @@
       <publish_visual_pose>false</publish_visual_pose>
       <publish_nested_model_pose>false</publish_nested_model_pose>
-      <update_frequency>50</update_frequency>
+      <update_frequency>100</update_frequency>  <!-- raised from 50: better MPC state feedback -->
     </plugin>
   </gazebo>
@@ -1846,6 +1854,6 @@
     <plugin filename="gz-sim-odometry-publisher-system"
             name="gz::sim::systems::OdometryPublisher">
-      <odom_frame>odom</odom_frame>
-      <robot_base_frame>base_link</robot_base_frame>
+      <odom_frame>${(ns + '/odom') if ns else 'odom'}</odom_frame>
+      <robot_base_frame>${(ns + '/base_link') if ns else 'base_link'}</robot_base_frame>
       <publish_rate>50</publish_rate>
     </plugin>
@@ -1861,5 +1869,5 @@
       <timeConstantUp>0.0125</timeConstantUp>
       <timeConstantDown>0.025</timeConstantDown>
-      <maxRotVelocity>1000.0</maxRotVelocity>
+      <maxRotVelocity>838.0</maxRotVelocity>  <!-- 838 rad/s → hover at ~75% throttle, max 1.75× hover thrust -->
       <motorConstant>1.740e-05</motorConstant>
       <momentConstant>0.01408</momentConstant>
@@ -1883,5 +1891,5 @@
       <timeConstantUp>0.0125</timeConstantUp>
       <timeConstantDown>0.025</timeConstantDown>
-      <maxRotVelocity>1000.0</maxRotVelocity>
+      <maxRotVelocity>838.0</maxRotVelocity>  <!-- 838 rad/s → hover at ~75% throttle, max 1.75× hover thrust -->
       <motorConstant>1.740e-05</motorConstant>
       <momentConstant>0.01408</momentConstant>
@@ -1905,5 +1913,5 @@
       <timeConstantUp>0.0125</timeConstantUp>
       <timeConstantDown>0.025</timeConstantDown>
-      <maxRotVelocity>1000.0</maxRotVelocity>
+      <maxRotVelocity>838.0</maxRotVelocity>  <!-- 838 rad/s → hover at ~75% throttle, max 1.75× hover thrust -->
       <motorConstant>1.740e-05</motorConstant>
       <momentConstant>0.01408</momentConstant>
@@ -1927,5 +1935,5 @@
       <timeConstantUp>0.0125</timeConstantUp>
       <timeConstantDown>0.025</timeConstantDown>
-      <maxRotVelocity>1000.0</maxRotVelocity>
+      <maxRotVelocity>838.0</maxRotVelocity>  <!-- 838 rad/s → hover at ~75% throttle, max 1.75× hover thrust -->
       <motorConstant>1.740e-05</motorConstant>
       <momentConstant>0.01408</momentConstant>
@@ -1949,5 +1957,5 @@
       <timeConstantUp>0.0125</timeConstantUp>
       <timeConstantDown>0.025</timeConstantDown>
-      <maxRotVelocity>1000.0</maxRotVelocity>
+      <maxRotVelocity>838.0</maxRotVelocity>  <!-- 838 rad/s → hover at ~75% throttle, max 1.75× hover thrust -->
       <motorConstant>1.740e-05</motorConstant>
       <momentConstant>0.01408</momentConstant>
@@ -1971,5 +1979,5 @@
       <timeConstantUp>0.0125</timeConstantUp>
       <timeConstantDown>0.025</timeConstantDown>
-      <maxRotVelocity>1000.0</maxRotVelocity>
+      <maxRotVelocity>838.0</maxRotVelocity>  <!-- 838 rad/s → hover at ~75% throttle, max 1.75× hover thrust -->
       <motorConstant>1.740e-05</motorConstant>
       <momentConstant>0.01408</momentConstant>
